File: 411 PCB/411 PCB Arduino + Board Design.kicad_sch (KiCad schematic)
At the start: 1 part, among them U1 ATmega328P-P

Commit message: Add files via upload
Parts:
- added C1, C2: 20p, symbol Device:C
- added C3, C4, C5: 100n, symbol Device:C
- added C6, C7: 1uF, symbol Device:C
- added D1: LED, symbol Device:LED
- added J1: ICSP CONN, symbol Connector:Conn_PIC_ICSP_ICD
- added J2: Conn_01x06_MountingPin, symbol Connector_Generic_MountingPin:Conn_01x06_MountingPin
- added J3: Conn_01x07, symbol Connector_Generic:Conn_01x07
- added J4: Conn_01x04, symbol Connector_Generic:Conn_01x04
- added J5: ~, symbol Regulator_Linear:AP2120-3.3
- added Q1: Q_NMOS_GDS, symbol Device:Q_NMOS_GDS
- added R1, R3: 10k, symbol Device:R
- added R2, R4, R5: 1k, symbol Device:R
- added SW1: SW_SPST, symbol Switch:SW_SPST
- added TP1, TP2, TP3, TP4: TestPoint, symbol Connector:TestPoint
- added Y1: 8 MHz, symbol Device:Crystal
Connections:
- net at U1.1 (~{RESET}/PC6): now also J1.5 (~{RST}), R1.2, SW1.2 (B), TP1.1
- net at U1.10 (XTAL2/PB7): now also C1.2, Y1.2
- net at U1.17 ((MOSI)PB3): now also J1.4 (MOSI)
- net at U1.18 ((MISO)PB4): now also J1.1 (MISO)
- net at U1.19 ((SCK)PB5): now also J1.3 (SCK), Q1.1 (G), R3.1
- net at U1.2 ((RXD)PD0): now also R4.1
- net +3.3V: now reaches U1.20 (AVCC)
- net +3.3V: now also U1.7 (VCC), C3.2, C4.2, C7.1, J3.3 (Pin_3), J4.2 (Pin_2), J5.2 (VOUT), R1.1, R2.1
- net at U1.21 (AREF): now also C5.2
- net GND: now reaches U1.22 (GND)
- net GND: now also U1.8 (GND), C1.1, C2.1, C3.1, C4.1, C5.1, C6.2, C7.2, J1.6 (GND), J2.1 (Pin_1), J3.2 (Pin_2), J4.1 (Pin_1), J5.3 (GND), Q1.3 (S), R3.2, SW1.1 (A)
- net at U1.27 ((ADC4/SDA)PC4): now also J3.5 (Pin_5), J4.4 (Pin_4)
- net at U1.28 ((ADC5/SCL)PC5): now also J3.4 (Pin_4), J4.3 (Pin_3)
- net at U1.3 ((TXD)PD1): now also R5.1
- net at U1.9 (XTAL1/PB6): now also C2.2, Y1.1
- new net: J2.5 (Pin_5), R5.2, TP4.1
- new net: J2.4 (Pin_4), R4.2, TP3.1
- new net: D1.1 (K), Q1.2 (D)
- new net: D1.2 (A), R2.2
- new net: J2.3 (Pin_3), TP2.1
- new net +5V: J1.2 (VCC)
- new net +VDC: C6.1, J5.1 (VIN)
Other:
- note added: "Battary input voltage of (TBD)"
- note added: "Clock LED Indicator (TBD mosfet part # and LED part #)"
- note added: "Color Sensor TCS-34725 (PLACE HOLDER PINOUT)"
- note added: "ICSP Connector to program the ATmega328P-P chip"
- note added: "OLED Display 128x32 SSD1306 (Place Holder)"
- note added: "USB to Serial Connector (to be determined part #)"
- note added: "Voltage Regulator powered by battery. +3.3V output voltage. Part # AP2120-3.3"
