File: 411 PCB.REV1/411 PCB Arduino + Board Design.kicad_pcb (KiCad board)
At the start: 2 copper layers, 28 parts, among them J1 ICSP CONN, J2 Conn_01x06_MountingPin, J4 Conn_01x04, Q1 Q_NMOS_GDS, SW1 SW_SPST, SW3 SW_MEC_5E, U1 ATmega328P-P, Y1 8 MHz

Commit message: Add files via upload
Parts:
- C1, C2, C3, C4, C5, C6, C7: footprint Capacitor_SMD:CP_Elec_4x3 -> Capacitor_SMD:C_0603_1608Metric_Pad1.08x0.95mm_HandSolder
- D1: footprint LED_THT:LED_D5.0mm_Horizontal_O6.35mm_Z15.0mm -> LED_THT:LED_D5.0mm_Clear
- J1: footprint Connector_Harwin:Harwin_LTek-Male_2x03_P2.00mm_Vertical -> Connector_PinHeader_1.00mm:PinHeader_2x03_P1.00mm_Vertical
- J4: footprint Arduino.display:Adafruit_SSD1306 -> Connector_PinHeader_1.00mm:PinHeader_1x04_P1.00mm_Vertical
- JP1: footprint Connector_PinHeader_1.00mm:PinHeader_1x07_P1.00mm_Vertical -> Connector_PinHeader_1.27mm:PinHeader_1x07_P1.27mm_Vertical
- Q1: footprint Connector:FanPinHeader_1x03_P2.54mm_Vertical -> Package_TO_SOT_THT:TO-92_Wide
- SW1: footprint Button_Switch_THT:SW_Slide_1P2T_CK_OS102011MS2Q -> Button_Switch_THT:SW_Tactile_Straight_KSA0Axx1LFTR
- TP1, TP2, TP3, TP4: footprint MountingHole:MountingHole_2.1mm -> Connector_PinHeader_1.00mm:PinHeader_1x01_P1.00mm_Vertical
- Y1: footprint Connector:JWT_A3963_1x02_P3.96mm_Vertical -> Connector_PinHeader_1.00mm:PinHeader_1x02_P1.00mm_Vertical
- moved TP4 110.9 mm to (144.8, 73.7)
- moved TP2 103.8 mm to (144.8, 68.6)
- moved TP3 102.2 mm to (154.9, 61.0)
- moved TP1 59.5 mm to (193.0, 66.0)
- moved J4 47.8 mm to (195.6, 95.0), turned to 180 degrees
- moved JP1 34.5 mm to (175.3, 68.6)
- moved C6 20.3 mm to (119.4, 42.3)
- moved J1 19.6 mm to (184.4, 69.6), turned to 90 degrees
- moved J5 18.5 mm to (127.0, 38.1), turned to -90 degrees
- moved C7 15.3 mm to (137.2, 41.5), turned to -90 degrees
- moved C1 12.8 mm to (145.6, 91.4)
- moved C2 11.4 mm to (146.5, 88.9)
- moved R1 9.48 mm to (157.5, 52.3)
- moved Y1 9.31 mm to (152.4, 88.9)
- moved SW1 6.47 mm to (142.2, 55.9), turned to 90 degrees
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Connections:
- SW3 pad 2: Net-(R6-Pad2) -> +3.3V
Routing:
- net GND: track 6.87 -> 0.00 mm
- net Net-(J2-Pin_4): track 2.06 -> 0.00 mm
- net Net-(U1-(RXD)PD0): track 1.37 -> 0.00 mm
- net Net-(J2-Pin_5): track 1.30 -> 0.00 mm
- net Net-(U1-(TXD)PD1): track 1.12 -> 0.00 mm

Commit message: Add files via upload
Parts:
- C1, C2, C3, C4, C5, C6, C7: footprint Capacitor_SMD:C_0603_1608Metric_Pad1.08x0.95mm_HandSolder -> Capacitor_SMD:C_1206_3216Metric_Pad1.33x1.80mm_HandSolder
- D1: footprint LED_THT:LED_D5.0mm_Clear -> LED_SMD:LED_0805_2012Metric_Pad1.15x1.40mm_HandSolder
- J5: footprint Connector:FanPinHeader_1x03_P2.54mm_Vertical -> Package_TO_SOT_SMD:SOT-23
- Q1: footprint Package_TO_SOT_THT:TO-92_Wide -> Package_TO_SOT_SMD:SOT-323_SC-70_Handsoldering
- SW1: footprint Button_Switch_THT:SW_Tactile_Straight_KSA0Axx1LFTR -> Button_Switch_THT:SW_PUSH_6mm
- SW3: footprint Button_Switch_THT:SW_PUSH_6mm_H4.3mm -> Button_Switch_SMD:SW_DIP_SPSTx03_Slide_9.78x9.8mm_W8.61mm_P2.54mm
- Y1: footprint Connector_PinHeader_1.00mm:PinHeader_1x02_P1.00mm_Vertical -> footprints:ATS08A-E_CTS
- moved Y1 83.6 mm to (68.8, 88.9)
- moved C2 80.1 mm to (67.0, 99.1)
- moved C1 70.8 mm to (75.2, 99.1)
- moved C3 56.2 mm to (172.7, 136.2)
- moved C5 53.7 mm to (162.6, 136.2), turned to 90 degrees
- moved R6 52.4 mm to (208.3, 137.2), turned to -90 degrees
- moved SW3 38.5 mm to (207.5, 124.5), turned to 90 degrees
- moved Q1 30.6 mm to (200.7, 43.2)
- moved J4 27.3 mm to (213.4, 74.2), turned to 0 degrees
- moved JP1 25.9 mm to (200.7, 73.7)
- moved R3 25.9 mm to (199.2, 50.8)
- moved SW1 18.8 mm to (158.1, 45.7)
- moved R4 18.4 mm to (138.2, 73.2)
- moved TP2 18.4 mm to (127.0, 73.2)
- moved TP3 18.4 mm to (137.2, 65.6)
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Connections:
- SW3 pad 2: +3.3V -> Net-(R6-Pad2)
- SW3 pad 3: Net-(R6-Pad2) -> unconnected-(SW3-K-Pad3)
- SW3 pad 4: Net-(R6-Pad2) -> Net-(SW3-A)
Routing:
- net Net-(U1-AREF): track 1.12 -> 0.00 mm
- net GND: track 0.00 -> 1.12 mm

Commit message: Updated Folder Layout
Newest PCB update
Changed lines of the file:
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@@
     (property "ki_keywords" "LED diode")
     (attr smd)
-    (fp_text reference "D1" (at 0 -1.65) (layer "F.SilkS")
+    (fp_text reference "D1" (at 0 -2.54) (layer "F.SilkS")
         (effects (font (size 1 1) (thickness 0.15)))
     )
-    (fp_text value "LED" (at 0 1.65) (layer "F.Fab")
+    (fp_text value "LED" (at 0 2.54) (layer "F.Fab")
         (effects (font (size 1 1) (thickness 0.15)))
     )
-    (fp_text user "${REFERENCE}" (at 0 0) (layer "F.Fab")
-        (effects (font (size 0.5 0.5) (thickness 0.08)))
-    )
-    (fp_line (start -1.86 -0.96) (end -1.86 0.96)
-      (stroke (width 0.12) (type solid)) (layer "F.SilkS"))
-    (fp_line (start -1.86 0.96) (end 1 0.96)
-      (stroke (width 0.12) (type solid)) (layer "F.SilkS"))
-    (fp_line (start 1 -0.96) (end -1.86 -0.96)
-      (stroke (width 0.12) (type solid)) (layer "F.SilkS"))
-    (fp_line (start -1.85 -0.95) (end 1.85 -0.95)
-      (stroke (width 0.05) (type solid)) (layer "F.CrtYd"))
-    (fp_line (start -1.85 0.95) (end -1.85 -0.95)
-      (stroke (width 0.05) (type solid)) (layer "F.CrtYd"))
-    (fp_line (start 1.85 -0.95) (end 1.85 0.95)
-      (stroke (width 0.05) (type solid)) (layer "F.CrtYd"))
-    (fp_line (start 1.85 0.95) (end -1.85 0.95)
-      (stroke (width 0.05) (type solid)) (layer "F.CrtYd"))
-    (fp_line (start -1 -0.3) (end -1 0.6)
-      (stroke (width 0.1) (type solid)) (layer "F.Fab"))
-    (fp_line (start -1 0.6) (end 1 0.6)
-      (stroke (width 0.1) (type solid)) (layer "F.Fab"))
-    (fp_line (start -0.7 -0.6) (end -1 -0.3)
-      (stroke (width 0.1) (type solid)) (layer "F.Fab"))
-    (fp_line (start 1 -0.6) (end -0.7 -0.6)
-      (stroke (width 0.1) (type solid)) (layer "F.Fab"))
-    (fp_line (start 1 0.6) (end 1 -0.6)
-      (stroke (width 0.1) (type solid)) (layer "F.Fab"))
-    (pad "1" smd roundrect (at -1.025 0) (size 1.15 1.4) (layers "F.Cu" "F.Paste" "F.Mask") (roundrect_rratio 0.217391)
-      (net 7 "Net-(D1-K)") (pinfunction "K") (pintype "passive"))
-    (pad "2" smd roundrect (at 1.025 0) (size 1.15 1.4) (layers "F.Cu" "F.Paste" "F.Mask") (roundrect_rratio 0.217391)
-      (net 8 "Net-(D1-A)") (pinfunction "A") (pintype "passive"))
+    (fp_rect (start -1.75 -1.4) (end 1.75 1.4)
+      (stroke (width 0.1) (type default)) (fill none) (layer "B.Fab"))
+    (pad "1" smd roundrect (at -1.403 0) (size 1.65 2.41) (layers "F.Cu" "F.Paste" "F.Mask") (roundrect_rratio 0.25)
+      (net 7 "Net-(D1-K)") (pinfunction "K") (pintype "passive") (thermal_bridge_angle 45))
+    (pad "2" smd roundrect (at 1.397 0) (size 1.65 2.41) (layers "F.Cu" "F.Paste" "F.Mask") (roundrect_rratio 0.25)
+      (net 8 "Net-(D1-A)") (pinfunction "A") (pintype "passive") (thermal_bridge_angle 45))
     (model "${KICAD6_3DMODEL_DIR}/LED_SMD.3dshapes/LED_0805_2012Metric.wrl"
       (offset (xyz 0 0 0))

Commit message: Updated PCB Layout
Parts:
- SW3: footprint Button_Switch_SMD:SW_DIP_SPSTx03_Slide_9.78x9.8mm_W8.61mm_P2.54mm -> Button_Switch_THT:SW_PUSH_6mm
- moved Y1 85.6 mm to (154.2, 93.4), turned to -90 degrees
- moved C6 81.9 mm to (161.5, 112.6), turned to 0 degrees
- moved C2 81.2 mm to (148.0, 93.4)
- moved R6 79.3 mm to (142.7, 92.7), turned to 90 degrees
- moved J5 77.6 mm to (154.9, 110.5), turned to 180 degrees
- moved R2 74.6 mm to (174.5, 109.7), turned to 0 degrees
- moved SW3 74.2 mm to (147.4, 81.0), turned to -90 degrees
- moved C7 72.8 mm to (161.5, 108.9), turned to 0 degrees
- moved C1 72.7 mm to (147.9, 98.3)
- moved Q1 63.1 mm to (174.2, 100.4)
- moved D1 63.0 mm to (174.4, 105.5)
- moved C3 54.5 mm to (154.5, 84.8), turned to 0 degrees
- moved C5 53.9 mm to (173.0, 83.3), turned to 180 degrees
- moved R3 51.8 mm to (174.0, 96.1)
- moved TP1 39.3 mm to (175.7, 91.5)
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Connections:
- U1 pad 12: /LED_EN -> unconnected-(U1-(AIN0)PD6-Pad12)
- U1 pad 13: Net-(SW3-A) -> unconnected-(U1-(AIN1)PD7-Pad13)
- U1 pad 5: unconnected-(U1-(INT1)PD3-Pad5) -> /LED_EN
- U1 pad 6: unconnected-(U1-(T0)PD4-Pad6) -> Net-(SW3-A)
Other:
- board outline added: 42.1 x 62.6 mm

Commit message: update
Parts:
- moved R3 1.90 mm to (175.9, 96.4)
- moved C5 1.63 mm to (173.1, 81.7)
- moved R6 1.34 mm to (141.5, 93.3)
- moved C2 1.26 mm to (147.3, 92.3)
- moved R2 1.12 mm to (173.7, 110.4)
- moved C7 0.99 mm to (161.9, 108.0)
- moved C1 0.95 mm to (147.0, 98.7)
- moved R1 0.87 mm to (165.5, 56.7), turned to 180 degrees
- moved D1 0.87 mm to (173.8, 106.0)
- moved Q1 0.52 mm to (173.7, 100.6)
- moved C4 0.46 mm to (173.0, 86.0)
- moved C6 0.37 mm to (161.9, 112.6)
Routing:
- net Net-(J1-~{RST}): track 0.00 -> 121.0 mm
- net +3.3V: track 0.00 -> 119.7 mm
- net /LED_EN: track 0.00 -> 45.1 mm
- net Net-(J1-SCK): track 0.00 -> 25.3 mm
- net Net-(SW3-A): track 0.00 -> 18.1 mm
- net Net-(U1-XTAL2/PB7): track 0.00 -> 15.9 mm
- net Net-(U1-XTAL1/PB6): track 0.00 -> 13.5 mm
- net Net-(J2-Pin_4): track 0.00 -> 9.28 mm
- net /SDA_3.3V: track 0.00 -> 9.16 mm
- net /SCL_3.3V: track 0.00 -> 8.78 mm
- net Net-(J2-Pin_5): track 0.00 -> 7.65 mm
- net Net-(J1-MOSI): track 0.00 -> 7.21 mm
- net Net-(U1-AREF): track 0.00 -> 6.55 mm
- net +VDC: track 0.00 -> 5.40 mm
- net Net-(R6-Pad2): track 0.00 -> 4.94 mm
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
Commit message: update
Parts:
- C1, C2, C3, C4, C5, C6, C7: footprint Capacitor_SMD:C_1206_3216Metric_Pad1.33x1.80mm_HandSolder -> Capacitor_SMD:C_0603_1608Metric_Pad1.08x0.95mm_HandSolder
- D1: footprint LED_SMD:LED_0805_2012Metric_Pad1.15x1.40mm_HandSolder -> LED_THT:LED_D5.0mm_Clear
- J5: footprint Package_TO_SOT_SMD:SOT-23 -> Connector:FanPinHeader_1x03_P2.54mm_Vertical
- Q1: footprint Package_TO_SOT_SMD:SOT-323_SC-70_Handsoldering -> Package_TO_SOT_THT:TO-92_Wide
- SW1: footprint Button_Switch_THT:SW_PUSH_6mm -> Button_Switch_THT:SW_Tactile_Straight_KSA0Axx1LFTR
- SW3: footprint Button_Switch_THT:SW_PUSH_6mm -> Button_Switch_THT:SW_PUSH_6mm_H4.3mm
- Y1: footprint footprints:ATS08A-E_CTS -> Connector_PinHeader_1.00mm:PinHeader_1x02_P1.00mm_Vertical
- moved C6 82.1 mm to (119.4, 42.3), turned to -90 degrees
- moved J5 77.6 mm to (127.0, 38.1), turned to -90 degrees
- moved R2 75.6 mm to (208.3, 43.2), turned to 90 degrees
- moved C7 70.9 mm to (137.2, 41.5), turned to -90 degrees
- moved D1 63.8 mm to (205.7, 50.8)
- moved Q1 39.9 mm to (203.2, 73.7)
- moved SW3 37.7 mm to (172.0, 109.5), turned to 0 degrees
- moved J4 34.4 mm to (195.6, 95.0), turned to 180 degrees
- moved TP1 30.9 mm to (193.0, 66.0)
- moved R6 28.7 mm to (161.1, 114.3), turned to 0 degrees
- moved R3 27.2 mm to (194.1, 76.2)
- moved J1 25.7 mm to (184.4, 69.6), turned to 90 degrees
- moved SW1 14.4 mm to (142.2, 55.9)
- moved TP3 13.5 mm to (154.9, 61.0)
- moved R1 9.20 mm to (157.5, 52.3), turned to -90 degrees
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Connections:
- SW3 pad 2: Net-(R6-Pad2) -> +3.3V
- SW3 pad 3: unconnected-(SW3-K-Pad3) -> Net-(R6-Pad2)
- SW3 pad 4: Net-(SW3-A) -> Net-(R6-Pad2)
- U1 pad 12: unconnected-(U1-(AIN0)PD6-Pad12) -> /LED_EN
- U1 pad 13: unconnected-(U1-(AIN1)PD7-Pad13) -> Net-(SW3-A)
- U1 pad 5: /LED_EN -> unconnected-(U1-(INT1)PD3-Pad5)
- U1 pad 6: Net-(SW3-A) -> unconnected-(U1-(T0)PD4-Pad6)
Routing:
- net Net-(J1-~{RST}): track 121.0 -> 0.00 mm
- net +3.3V: track 119.7 -> 0.07 mm
- net /LED_EN: track 45.1 -> 0.00 mm
- net Net-(J1-SCK): track 25.3 -> 0.00 mm
- net Net-(SW3-A): track 18.1 -> 0.00 mm
- net Net-(U1-XTAL2/PB7): track 15.9 -> 0.00 mm
- net Net-(U1-XTAL1/PB6): track 13.5 -> 0.00 mm
- net Net-(J2-Pin_4): track 9.28 -> 0.00 mm
- net /SDA_3.3V: track 9.16 -> 0.00 mm
- net /SCL_3.3V: track 8.78 -> 0.00 mm
- net Net-(J2-Pin_5): track 7.65 -> 0.00 mm
- net Net-(J1-MOSI): track 7.21 -> 0.00 mm
- net Net-(U1-AREF): track 6.55 -> 1.12 mm
- net +VDC: track 5.40 -> 0.00 mm
- net Net-(R6-Pad2): track 4.94 -> 0.00 mm
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Other:
- board outline removed
