File: 411 PCB.REV2/411 PCB Arduino + Board Design.kicad_pcb (KiCad board)
At the start: 2 copper layers, 42.1 x 62.6 mm, 28 parts, among them J1 ICSP CONN, J2 Conn_01x06_MountingPin, J4 Conn_01x04, Q1 Q_NMOS_GDS, SW1 SW_SPST, SW3 SW_MEC_5E, U1 ATmega328P-P, Y1 8 MHz

Commit message: update
Parts:
- added TP5: TestPoint, Connector_PinHeader_1.00mm:PinHeader_1x01_P1.00mm_Vertical, F.Cu at (175.9, 67.9)
- added TP6: TestPoint, Connector_PinHeader_1.00mm:PinHeader_1x01_P1.00mm_Vertical, F.Cu at (175.8, 70.2)
- C1, C2: value 20p -> 10p
- D1: value LED -> LED (100mA Max)
- Y1: value 8 MHz -> 8 MHz
- moved J4 2.85 mm to (173.3, 66.8)
- moved JP1 1.43 mm to (170.5, 65.2)
Routing:
- net +3.3V: track 119.7 -> 117.0 mm
- net /LED_EN: track 45.1 -> 46.6 mm
