File: 411 PCB.REV3/411 PCB Arduino + Board Design.kicad_sch (KiCad schematic)
At the start: 35 parts, among them J1 ICSP CONN, J3 Conn_01x04, J4 HEADER-1X770MIL, Q1 Q_NMOS_GDS, SW1 SW_SPST, SW2 SW_MEC_5E, U2 ATmega328P-P, Y1 8 MHz

Commit message: 411 PCB Rev4+ Updated and Routed Layout
This is the pre submission board. Before Ben check
Parts:
- J3: footprint Connector_PinHeader_1.00mm:PinHeader_1x04_P1.00mm_Vertical -> Connector_PinHeader_2.54mm:PinHeader_1x04_P2.54mm_Vertical
- J4: footprint Connector_PinHeader_1.27mm:PinHeader_1x07_P1.27mm_Vertical -> Connector_PinHeader_2.54mm:PinHeader_1x07_P2.54mm_Vertical
- LED1: renamed from B_LED1; value LED (100mA Max) -> Blue LED (100mA Max)
- SW2: footprint Button_Switch_THT:SW_PUSH_6mm -> Connector_PinHeader_2.54mm:PinHeader_1x04_P2.54mm_Vertical
Connections:
- net SCL_3.3V renamed SDA-
- net SDA_3.3V renamed SDA+
Other:
- moved on the sheet: J3
Changed lines of the file:
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@@
     (effects (font (size 1.2446 1.2446)) (justify left bottom))
   )
-  (label "SDA_3.3V" (at 383.54 191.77 0) (fields_autoplaced)
+  (label "SDA+" (at 383.54 191.77 0) (fields_autoplaced)
     (effects (font (size 1.2446 1.2446)) (justify left bottom))
   )
@@
     (effects (font (size 1.2446 1.2446)) (justify left bottom))
   )
-  (label "SCL_3.3V" (at 383.54 189.23 0) (fields_autoplaced)
+  (label "SDA-" (at 383.54 189.23 0) (fields_autoplaced)
     (effects (font (size 1.2446 1.2446)) (justify left bottom))
   )
@@
       (effects (font (size 1.27 1.27)))
     )
-    (property "Footprint" "Button_Switch_THT:SW_PUSH_6mm" (at 215.9 204.47 0)
+    (property "Footprint" "Connector_PinHeader_2.54mm:PinHeader_1x04_P2.54mm_Vertical" (at 215.9 204.47 0)
       (effects (font (size 1.27 1.27)) hide)
     )
@@
       (effects (font (size 1.778 1.5113)) (justify left bottom) hide)
     )
-    (property "Footprint" "Connector_PinHeader_1.27mm:PinHeader_1x07_P1.27mm_Vertical" (at 392.43 173.99 0)
+    (property "Footprint" "Connector_PinHeader_2.54mm:PinHeader_1x07_P2.54mm_Vertical" (at 392.43 173.99 0)
       (effects (font (size 1.27 1.27)) hide)
     )
@@
   (symbol (lib_id "Device:LED") (at 397.51 223.52 90) (unit 1)
     (in_bom yes) (on_board yes) (dnp no)
-    (property "Reference" "B_LED1" (at 401.32 224.79 90)
+    (property "Reference" "LED1" (at 401.32 224.79 90)
       (effects (font (size 1.27 1.27)) (justify right))
     )
-    (property "Value" "LED (100mA Max)" (at 377.19 224.79 90)
+    (property "Value" "Blue LED (100mA Max)" (at 374.65 224.79 90)
       (effects (font (size 1.27 1.27)) (justify right))
     )
@@
       (project "411 PCB Arduino + Board Design"
         (path "/3b213592-ad28-4b80-bc7a-214b9fe026d8"
-          (reference "B_LED1") (unit 1)
+          (reference "LED1") (unit 1)
         )
       )
@@
       (effects (font (size 1.27 1.27)) (justify left) hide)
     )
-    (property "Footprint" "Connector_PinHeader_1.00mm:PinHeader_1x04_P1.00mm_Vertical" (at 341.63 158.75 0)
-      (effects (font (size 1.27 1.27)) hide)
-    )
+    (property "Footprint" "Connector_PinHeader_2.54mm:PinHeader_1x04_P2.54mm_Vertical" (at 341.63 158.75 0)
+      (effects (font (size 1.27 1.27)) hide)
+    )
