File: 411 PCB.REV4/411 PCB Arduino + Board Design.kicad_sch (KiCad schematic)
At the start: 37 parts, among them J1 ICSP CONN, J3 Conn_01x04, J4 Conn_01x05_Pin, Q1 Q_NMOS_GDS, SW1 SW_SPST, SW2 SW_MEC_5E, SW3 SW_SPDT, SW4 SW_DPST_x2, U2 ATmega328P-P, Y1 8 MHz

Commit message: Updated Board + PCB purchase receipt
Yes
Connections:
- no-connect marks 11 -> 12
Other:
- note added: "Power module connecting with VBUS (+) and -GND (-)"
- note added: "Programmer switch: In 5V state the chip allowes us to program it . If 3.3V switch then the chip is in active mode."
- title: Color Sensor -> Color Sensor (Team 3)
- moved on the sheet: SW3A
Changed lines of the file:
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@@
   (paper "A2")
   (title_block
-    (title "Color Sensor")
+    (title "Color Sensor (Team 3)")
     (date "2023-11-14")
-    (rev "3")
+    (rev "4")
   )
   (junction (at 279.4 260.35) (diameter 0) (color 0 0 0 0)
@@
   (junction (at 261.62 189.23) (diameter 0) (color 0 0 0 0)
   )
-  (junction (at 334.01 204.47) (diameter 0) (color 0 0 0 0)
-  )
   (junction (at 243.84 226.06) (diameter 0) (color 0 0 0 0)
   )
@@
   )
   (junction (at 325.12 189.23) (diameter 0) (color 0 0 0 0)
+  )
+  (junction (at 334.01 205.74) (diameter 0) (color 0 0 0 0)
   )
   (junction (at 168.91 96.52) (diameter 0) (color 0 0 0 0)
@@
   (no_connect (at 267.97 240.03))
   (no_connect (at 298.45 247.65))
+  (no_connect (at 220.98 215.9))
   (no_connect (at 267.97 237.49))
   (no_connect (at 298.45 245.11))
@@
     (stroke (width 0) (type default))
   )
-  (wire (pts (xy 275.59 135.89) (xy 281.94 135.89))
+  (wire (pts (xy 316.23 135.89) (xy 309.88 135.89))
     (stroke (width 0) (type default))
   )
@@
     (stroke (width 0) (type default))
   )
-  (wire (pts (xy 304.8 132.08) (xy 304.8 133.35))
+  (wire (pts (xy 287.02 132.08) (xy 287.02 133.35))
     (stroke (width 0) (type default))
   )
@@
     (stroke (width 0) (type default))
   )
-  (wire (pts (xy 292.1 133.35) (xy 304.8 133.35))
+  (wire (pts (xy 299.72 133.35) (xy 287.02 133.35))
     (stroke (width 0) (type default))
   )
@@
     (stroke (width 0) (type default))
   )
-  (wire (pts (xy 314.96 132.08) (xy 314.96 138.43))
+  (wire (pts (xy 276.86 132.08) (xy 276.86 138.43))
     (stroke (width 0) (type default))
   )
@@
     (stroke (width 0) (type default))
   )
-  (wire (pts (xy 334.01 204.47) (xy 365.76 204.47))
+  (wire (pts (xy 334.01 205.74) (xy 365.76 205.74))
     (stroke (width 0) (type default))
   )
@@
     (stroke (width 0) (type default))
   )
-  (wire (pts (xy 275.59 133.35) (xy 275.59 135.89))
+  (wire (pts (xy 316.23 133.35) (xy 316.23 135.89))
     (stroke (width 0) (type default))
   )
@@
     (stroke (width 0) (type default))
   )
-  (wire (pts (xy 314.96 138.43) (xy 292.1 138.43))
+  (wire (pts (xy 276.86 138.43) (xy 299.72 138.43))
     (stroke (width 0) (type default))
   )
@@
     (stroke (width 0) (type default))
   )
-  (wire (pts (xy 365.76 204.47) (xy 365.76 194.31))
+  (wire (pts (xy 365.76 205.74) (xy 365.76 194.31))
     (stroke (width 0) (type default))
   )
@@
     (fill (type none))
   )
+  (rectangle (start 78.74 91.44) (end 93.98 120.65)
+    (stroke (width 0) (type default))
+    (fill (type none))
+  )
+  (rectangle (start 269.24 118.11) (end 321.31 146.05)
+    (stroke (width 0) (type default))
+    (fill (type none))
+  )
   (rectangle (start 322.58 154.94) (end 370.84 186.69)
     (stroke (width 0) (type default))
@@
     (fill (type none))
   )
-  (rectangle (start 72.39 58.42) (end 193.04 137.16)
+  (rectangle (start 58.42 58.42) (end 193.04 137.16)
     (stroke (width 0) (type default))
     (fill (type none))
@@
   )
   (text "Switch Push Button\nChanges the state of device" (at 203.2 223.52 0)
+    (effects (font (size 1.27 1.27)) (justify left bottom))
+  )
+  (text "Power module connecting with VBUS (+) and -GND (-)\n"
+    (at 58.42 123.19 0)
+    (effects (font (size 1.27 1.27)) (justify left bottom))
+  )
+  (text "Programmer switch: In 5V state the chip allowes us to program it\n. If 3.3V switch then the chip is in active mode."
+    (at 265.43 116.84 0)
     (effects (font (size 1.27 1.27)) (justify left bottom))
   )
@@
     )
   )
-  (symbol (lib_id "power:VCC") (at 275.59 133.35 0) (unit 1)
-    (in_bom yes) (on_board yes) (dnp no) (fields_autoplaced)
-    (property "Reference" "#PWR03" (at 275.59 137.16 0)
-      (effects (font (size 1.27 1.27)) hide)
-    )
-    (property "Value" "VCC" (at 275.59 128.27 0)
-      (effects (font (size 1.27 1.27)))
-    )
-    (property "Footprint" "" (at 275.59 133.35 0)
-      (effects (font (size 1.27 1.27)) hide)
-    )
-    (property "Datasheet" "" (at 275.59 133.35 0)
+  (symbol (lib_id "power:VCC") (at 316.23 133.35 0) (mirror y) (unit 1)
+    (in_bom yes) (on_board yes) (dnp no) (fields_autoplaced)
+    (property "Reference" "#PWR03" (at 316.23 137.16 0)
+      (effects (font (size 1.27 1.27)) hide)
+    )
+    (property "Value" "VCC" (at 316.23 128.27 0)
+      (effects (font (size 1.27 1.27)))
+    )
+    (property "Footprint" "" (at 316.23 133.35 0)
+      (effects (font (size 1.27 1.27)) hide)
+    )
+    (property "Datasheet" "" (at 316.23 133.35 0)
       (effects (font (size 1.27 1.27)) hide)
     )
@@
     )
   )
-  (symbol (lib_id "power:+3.3V") (at 314.96 132.08 0) (unit 1)
-    (in_bom yes) (on_board yes) (dnp no)
-    (property "Reference" "#+3.3V01" (at 314.96 135.89 0)
-      (effects (font (size 1.27 1.27)) hide)
-    )
-    (property "Value" "+3.3V" (at 314.96 128.27 0)
-      (effects (font (size 1.27 1.27)))
-    )
-    (property "Footprint" "" (at 314.96 132.08 0)
-      (effects (font (size 1.27 1.27)) hide)
-    )
-    (property "Datasheet" "" (at 314.96 132.08 0)
+  (symbol (lib_id "power:+3.3V") (at 276.86 132.08 0) (mirror y) (unit 1)
+    (in_bom yes) (on_board yes) (dnp no)
+    (property "Reference" "#+3.3V01" (at 276.86 135.89 0)
+      (effects (font (size 1.27 1.27)) hide)
+    )
+    (property "Value" "+3.3V" (at 276.86 128.27 0)
+      (effects (font (size 1.27 1.27)))
+    )
+    (property "Footprint" "" (at 276.86 132.08 0)
+      (effects (font (size 1.27 1.27)) hide)
+    )
+    (property "Datasheet" "" (at 276.86 132.08 0)
       (effects (font (size 1.27 1.27)) hide)
     )
@@
     )
     (property "Value" "Conn_01x01_Pin" (at 83.82 119.38 0)
-      (effects (font (size 1.27 1.27)))
+      (effects (font (size 1.27 1.27)) hide)
     )
     (property "Footprint" "Connector_PinHeader_2.54mm:PinHeader_1x01_P2.54mm_Vertical" (at 85.09 116.84 0)
@@
     )
     (property "Value" "Conn_01x01_Pin" (at 76.2 101.6 0)
-      (effects (font (size 1.27 1.27)) (justify left))
+      (effects (font (size 1.27 1.27)) (justify left) hide)
     )
     (property "Footprint" "Connector_PinHeader_2.54mm:PinHeader_1x01_P2.54mm_Vertical" (at 85.09 99.06 0)
@@
     )
   )
-  (symbol (lib_id "Switch:SW_DPDT_x2") (at 287.02 135.89 0) (unit 1)
-    (in_bom yes) (on_board yes) (dnp no) (fields_autoplaced)
-    (property "Reference" "SW3" (at 287.02 128.27 0)
-      (effects (font (size 1.27 1.27)))
-    )
-    (property "Value" "SW_SPDT" (at 287.02 130.81 0)
-      (effects (font (size 1.27 1.27)))
-    )
-    (property "Footprint" "Button_Switch_THT:SW_E-Switch_EG1271_SPDT_123" (at 287.02 135.89 0)
-      (effects (font (size 1.27 1.27)) hide)
-    )
-    (property "Datasheet" "~" (at 287.02 135.89 0)
+  (symbol (lib_id "Switch:SW_DPDT_x2") (at 304.8 135.89 0) (mirror y) (unit 1)
+    (in_bom yes) (on_board yes) (dnp no) (fields_autoplaced)
+    (property "Reference" "SW3" (at 304.8 128.27 0)
+      (effects (font (size 1.27 1.27)))
+    )
+    (property "Value" "SW_SPDT" (at 304.8 130.81 0)
+      (effects (font (size 1.27 1.27)))
+    )
+    (property "Footprint" "Button_Switch_THT:SW_E-Switch_EG1271_SPDT_123" (at 304.8 135.89 0)
+      (effects (font (size 1.27 1.27)) hide)
+    )
+    (property "Datasheet" "~" (at 304.8 135.89 0)
       (effects (font (size 1.27 1.27)) hide)
     )
@@
     )
   )
-  (symbol (lib_name "+5V_1") (lib_id "power:+5V") (at 304.8 132.08 0) (unit 1)
-    (in_bom yes) (on_board yes) (dnp no)
-    (property "Reference" "#PWR09" (at 304.8 135.89 0)
-      (effects (font (size 1.27 1.27)) hide)
-    )
-    (property "Value" "+5V (Programmer Source)" (at 318.77 125.73 0)
+  (symbol (lib_name "+5V_1") (lib_id "power:+5V") (at 287.02 132.08 0) (mirror y) (unit 1)
+    (in_bom yes) (on_board yes) (dnp no)
+    (property "Reference" "#PWR09" (at 287.02 135.89 0)
+      (effects (font (size 1.27 1.27)) hide)
+    )
+    (property "Value" "+5V (Programmer Source)" (at 273.05 125.73 0)
       (effects (font (size 1.27 1.27)) (justify right))
     )
-    (property "Footprint" "" (at 304.8 132.08 0)
-      (effects (font (size 1.27 1.27)) hide)
-    )
-    (property "Datasheet" "" (at 304.8 132.08 0)
-      (effects (font (size 1.27 1.27)) hide)
-    )
+    (property "Footprint" "" (at 287.02 132.08 0)
+      (effects (font (size 1.27 1.27)) hide)
+    )
+    (property "Datasheet" "" (at 287.02 132.08 0)
+      (effects (font (size 1.27 1.27)) hide)
+    )
